File: hardware/CAN-RAMPS/CAN-RAMPS.sch (EAGLE design)
At the start: 31 parts, among them Q1 12MHZ, U1 MCP2515(MCP2510)ML, U2 MCP2551, U4 ATTINY816M

Commit message: Added mounting tabs
Parts:
- added H1, H2: MOUNT-PAD-ROUND3.2, holes:MOUNT-PAD-ROUND3.2
Connections:
- net GND: now also H1.MOUNT, H2.MOUNT
Changed lines of the file:
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@@
 <part name="+3V5" library="supply1" library_urn="urn:adsk.eagle:library:371" deviceset="+3V3" device=""/>
 <part name="J3" library="SparkFun-Connectors" library_urn="urn:adsk.eagle:library:513" deviceset="CONN_06" device="LOCK_LONGPADS" package3d_urn="urn:adsk.eagle:package:38121/1"/>
+<part name="H1" library="holes" library_urn="urn:adsk.eagle:library:237" deviceset="MOUNT-PAD-ROUND" device="3.2" package3d_urn="urn:adsk.eagle:package:14282/1"/>
+<part name="H2" library="holes" library_urn="urn:adsk.eagle:library:237" deviceset="MOUNT-PAD-ROUND" device="3.2" package3d_urn="urn:adsk.eagle:package:14282/1"/>
 </parts>
 <sheets>
@@
 <instance part="+3V5" gate="G$1" x="127" y="45.72"/>
 <instance part="J3" gate="G$1" x="233.68" y="93.98" rot="MR0"/>
+<instance part="H1" gate="G$1" x="30.48" y="45.72" rot="R180"/>
+<instance part="H2" gate="G$1" x="30.48" y="38.1" rot="R180"/>
 </instances>
 <busses>
@@
 <wire x1="38.1" y1="27.94" x2="40.64" y2="27.94" width="0.1524" layer="91"/>
 <pinref part="C7" gate="G$1" pin="2"/>
-<wire x1="38.1" y1="27.94" x2="38.1" y2="50.8" width="0.1524" layer="91"/>
+<wire x1="38.1" y1="27.94" x2="38.1" y2="38.1" width="0.1524" layer="91"/>
 <junction x="38.1" y="27.94"/>
-</segment>
-<segment>
+<pinref part="H1" gate="G$1" pin="MOUNT"/>
+<wire x1="38.1" y1="38.1" x2="38.1" y2="45.72" width="0.1524" layer="91"/>
+<wire x1="38.1" y1="45.72" x2="38.1" y2="50.8" width="0.1524" layer="91"/>
+<wire x1="33.02" y1="45.72" x2="38.1" y2="45.72" width="0.1524" layer="91"/>
+<junction x="38.1" y="45.72"/>
+<pinref part="H2" gate="G$1" pin="MOUNT"/>
+<wire x1="33.02" y1="38.1" x2="38.1" y2="38.1" width="0.1524" layer="91"/>
+<junction x="38.1" y="38.1"/>
+</segment>
+<segment>
